File: LoRa+GPS/PCB_LoRA+GPS.kicad_sch (KiCad schematic)
At the start: 66 parts, among them J1 Conn_Coaxial_Small, J2 USB_C_Receptacle_USB2.0_16P, J4 Conn_Coaxial_Small, Q2 SS8050, Q3 AO3400A, Q4 SS8050, SW1 SW_Push, U1 ESP32-PICO-D4, U2 RFM95W-915S2, U3 TPS62A01ADRL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

Commit message: Add files via upload
Parts:
- added SW2: SW_SPST, Button_Switch_THT:SW_E-Switch_EG1271_SPDT, symbol Switch:SW_SPST
- J1: footprint Connector_Coaxial:U.FL_Molex_MCRF_73412-0110_Vertical -> Connector_Coaxial:U.FL_Hirose_U.FL-R-SMT-1_Vertical
- SW1: footprint Button_Switch_SMD:SW_Push_1P1T_NO_Vertical_Wuerth_434133025816 -> Button_Switch_SMD:SW_Push_1P1T_NO_CK_KMR2
Connections:
- net +BATT: now also SW2.1 (A); no longer BT2.1 (+)
- new net: BT2.1 (+), SW2.2 (B)
Other:
- moved on the sheet: BT2
Changed lines of the file:
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@@
 	(text "R11 y R12 indican al usb que el dispositivo es sink\nR4 y R5 fueron elegidas para obtener 3.3V a la salida. R5 =< 100k (segun DS)\nC* es un cap opcional según datasheet"
 		(exclude_from_sim no)
-		(at 20.066 221.742 0)
+		(at 18.542 243.078 0)
 		(effects
 			(font
@@
 	)
 	(junction
-		(at 66.04 207.01)
+		(at 66.04 224.79)
 		(diameter 0)
 		(color 0 0 0 0)
@@
 	(wire
 		(pts
-			(xy 66.04 207.01) (xy 71.12 207.01)
+			(xy 66.04 224.79) (xy 71.12 224.79)
 		)
 		(stroke
@@
 	(wire
 		(pts
+			(xy 62.23 205.74) (xy 62.23 224.79)
+		)
+		(stroke
+			(width 0)
+			(type default)
+		)
+	)
+	(wire
+		(pts
 			(xy 289.56 53.34) (xy 279.4 53.34)
 		)
@@
 	(wire
 		(pts
-			(xy 71.12 207.01) (xy 71.12 204.47)
-		)
-		(stroke
-			(width 0)
-			(type default)
-		)
-	)
-	(wire
-		(pts
 			(xy 138.43 205.74) (xy 139.7 205.74)
 		)
@@
 	(wire
 		(pts
+			(xy 71.12 222.25) (xy 71.12 224.79)
+		)
+		(stroke
+			(width 0)
+			(type default)
+		)
+	)
+	(wire
+		(pts
 			(xy 293.37 109.22) (xy 297.18 109.22)
 		)
@@
 	(wire
 		(pts
-			(xy 66.04 208.28) (xy 66.04 207.01)
+			(xy 66.04 226.06) (xy 66.04 224.79)
 		)
 		(stroke
@@
 	(wire
 		(pts
-			(xy 62.23 207.01) (xy 66.04 207.01)
+			(xy 62.23 224.79) (xy 66.04 224.79)
 		)
 		(stroke
@@
 	(wire
 		(pts
+			(xy 71.12 207.01) (xy 71.12 214.63)
+		)
+		(stroke
+			(width 0)
+			(type default)
+		)
+	)
+	(wire
+		(pts
 			(xy 127 180.34) (xy 127 177.8)
 		)
@@
 	(wire
 		(pts
-			(xy 62.23 205.74) (xy 62.23 207.01)
-		)
-		(stroke
-			(width 0)
-			(type default)
-		)
-	)
-	(wire
-		(pts
 			(xy 279.4 48.26) (xy 264.16 48.26)
 		)
@@
 			)
 		)
-		(property "Footprint" "Button_Switch_SMD:SW_Push_1P1T_NO_Vertical_Wuerth_434133025816"
+		(property "Footprint" "Button_Switch_SMD:SW_Push_1P1T_NO_CK_KMR2"
 			(at 332.74 172.72 0)
 			(effects
@@
 	(symbol
 		(lib_id "power:GND")
-		(at 66.04 208.28 0)
+		(at 66.04 226.06 0)
 		(unit 1)
 		(exclude_from_sim no)
@@
 		(fields_autoplaced yes)
 		(property "Reference" "#PWR01"
-			(at 66.04 214.63 0)
+			(at 66.04 232.41 0)
 			(effects
 				(font
@@
 		)
 		(property "Value" "GND"
-			(at 66.04 213.36 0)
+			(at 66.04 231.14 0)
 			(effects
 				(font
@@
 		)
 		(property "Footprint" ""
-			(at 66.04 208.28 0)
+			(at 66.04 226.06 0)
 			(effects
 				(font
@@
 		)
 		(property "Datasheet" ""
-			(at 66.04 208.28 0)
+			(at 66.04 226.06 0)
 			(effects
 				(font
@@
 		)
 		(property "Description" "Power symbol creates a global label with name \"GND\" , ground"
-			(at 66.04 208.28 0)
+			(at 66.04 226.06 0)
 			(effects
 				(font
@@
 	(symbol
 		(lib_id "Device:Battery_Cell")
-		(at 71.12 201.93 0)
+		(at 71.12 219.71 0)
 		(unit 1)
 		(exclude_from_sim no)
@@
 		(fields_autoplaced yes)
 		(property "Reference" "BT2"
-			(at 74.93 198.8184 0)
+			(at 74.93 216.5984 0)
 			(effects
 				(font
@@
 		)
 		(property "Value" "Battery_Cell"
-			(at 74.93 201.3584 0)
+			(at 74.93 219.1384 0)
 			(effects
 				(font
@@
 		)
 		(property "Footprint" "Connector_JST:JST_EH_S2B-EH_1x02_P2.50mm_Horizontal"
-			(at 71.12 200.406 90)
+			(at 71.12 218.186 90)
 			(effects
 				(font
@@
 		)
 		(property "Datasheet" "~"
-			(at 71.12 200.406 90)
+			(at 71.12 218.186 90)
 			(effects
 				(font
@@
 		)
 		(property "Description" "Single-cell battery"
-			(at 71.12 201.93 0)
+			(at 71.12 219.71 0)
 			(effects
 				(font
@@
 			)
 		)
-		(property "Footprint" "Connector_Coaxial:U.FL_Molex_MCRF_73412-0110_Vertical"
+		(property "Footprint" "Connector_Coaxial:U.FL_Hirose_U.FL-R-SMT-1_Vertical"
 			(at 308.61 96.52 0)
 			(effects
@@
 					(unit 1)
 				)
+			)
+		)
+	)
+	(symbol
+		(lib_id "Switch:SW_SPST")
+		(at 71.12 201.93 270)
+		(unit 1)
+		(exclude_from_sim no)
+		(in_bom yes)
+		(on_board yes)
+		(dnp no)
+		(fields_autoplaced yes)
+		(property "Reference" "SW2"
+			(at 73.66 200.6599 90)
+			(effects
+				(font
+					(size 1.27 1.27)
+				)
+				(justify left)
+			)
+		)
+		(property "Value" "SW_SPST"
+			(at 73.66 203.1999 90)
+			(effects
+				(font
+					(size 1.27 1.27)
+				)
+				(justify left)
+			)
+		)
+		(property "Footprint" "Button_Switch_THT:SW_E-Switch_EG1271_SPDT"
+			(at 71.12 201.93 0)
+			(effects
+				(font
+					(size 1.27 1.27)
+				)
+				(hide yes)
+			)
+		)
+		(property "Datasheet" "~"
+			(at 71.12 201.93 0)
+			(effects
+				(font
+					(size 1.27 1.27)
+				)
+				(hide yes)
+			)
+		)
+		(property "Description" "Single Pole Single Throw (SPST) switch"
+			(at 71.12 201.93 0)
+			(effects
+				(font
+					(size 1.27 1.27)
+				)
+				(hide yes)
+			)
+		)
+		(pin "2"
+		)
+		(pin "1"
+		)
+		(instances
+			(project ""
+				(path "/80d6a340-3f89-493a-85f7-c642314f6a81"
+					(reference "SW2")
+					(unit 1)
+				)
