File: LoRa+GPS/PCB_LoRa+GPS.kicad_pcb (KiCad board)
At the start: 4 copper layers, 80 x 50 mm, 69 parts, among them J1 Conn_Coaxial_Small, J2 USB_C_Receptacle_USB2.0_16P, J4 Conn_Coaxial_Small, Q2 SS8050, Q3 AO3400A, Q4 SS8050, SW1 SW_Push, SW2 SW_SPST, U1 ESP32-PICO-D4, U2 RFM95W-915S2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

Commit message: V2 DRC checked
Parts:
- added Q1: AO3401A, Package_TO_SOT_SMD:SOT-23, B.Cu at (52.5, 53.5)
- added R26: 1k, Resistor_SMD:R_0402_1005Metric, B.Cu at (52.0, 50.5)
- added R27: 10k, Resistor_SMD:R_0402_1005Metric, B.Cu at (54.2, 50.5)
Connections:
- C20 pad 2: Net-(U5-VCC) -> Net-(Q1-S)
- L2 pad 2: Net-(U5-VCC) -> Net-(Q1-S)
- U5 pad 7: Net-(U5-VCC) -> Net-(Q1-D)
- U5 pad 8: Net-(U5-VCC) -> Net-(Q1-D)
Routing:
- net unconnected-(R26-Pad1): track 0.00 -> 20.3 mm, vias 0 -> 1
- net Net-(Q1-S): track 0.00 -> 11.8 mm, vias 0 -> 1
- net Net-(U5-VCC): track 9.22 -> 0.00 mm
- net GND: track 12.6 -> 21.1 mm, vias 59 -> 63
- net Net-(Q1-D): track 0.00 -> 8.50 mm, vias 0 -> 1
- net Rx_GPS: track 38.3 -> 40.6 mm
- net Pnp_Gps: track 0.00 -> 2.29 mm
- net USB_D-: track 13.2 -> 11.0 mm
- net 3V3: track 77.5 -> 79.4 mm
- net USB_D+: track 12.8 -> 11.0 mm
- net SCK_LoRa: track 40.8 -> 42.6 mm
- net Net-(D2-K): track 8.96 -> 7.32 mm
- net Reset_LoRa: track 55.1 -> 56.6 mm
- net TRIG_Sensor: track 11.4 -> 10.2 mm
- net Net-(Q4-E): track 31.4 -> 32.3 mm
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