File: LoRa+GPS/PCB_LoRa+GPS.kicad_pcb (KiCad board)
At the start: 4 copper layers, 80 x 50 mm, 84 parts, among them J1 Conn_Coaxial_Small, J2 USB_C_Receptacle_USB2.0_16P, J4 Conn_Coaxial_Small, Q1 AO3401A, Q2 SS8050, Q3 AO3400A, Q4 SS8050, SW1 SW_Push, SW2 SW_SPST, U1 ESP32-PICO-D4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

Commit message: Add files via upload
Routing:
- net 3V3: track 77.7 -> 81.1 mm, vias 7 -> 8
- net USB_D-: track 11.0 -> 12.7 mm
- net USB_D+: track 11.0 -> 12.7 mm
- net GND: track 24.0 -> 22.9 mm
