File: LoRa+GPS/PCB_LoRa+GPS.kicad_sch (KiCad schematic)
At the start: 67 parts, among them J1 Conn_Coaxial_Small, J2 USB_C_Receptacle_USB2.0_16P, J4 Conn_Coaxial_Small, Q2 SS8050, Q3 AO3400A, Q4 SS8050, SW1 SW_Push, SW2 SW_SPST, U1 ESP32-PICO-D4, U2 RFM95W-915S2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

Commit message: Add files via upload
Parts:
- added BT1: 1056TR, CR1220 socket:BAT_1056TR, symbol Battery_CR1220:1056TR
- added R25: 10k, Resistor_SMD:R_0402_1005Metric, symbol Device:R
Connections:
- net 3.3V is gone; now on net 3V3: R18.2
- net GND: now also J1.2 (Ext), BT1.N, R25.2; no longer J1.1 (In)
- net Wake_GPS: now reaches U1.20 (IO13)
- net Wake_GPS: now also U5.5 (Wake-Up)
- net AntOff_GPS: now reaches U1.42 (IO21)
- net AntOff_GPS: now also U5.13 (ANT_OFF), R25.1
- net at C20.2, L2.2, U5.7 (VCC_IO)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: no longer U5.6 (VBATT)
- net at U2.9 (ANT): now also J1.1 (In); no longer J1.2 (Ext)
- new net VBatt: BT1.P, U5.6 (VBATT)

Commit message: V2 DRC checked
Parts:
- added Q1: AO3401A, Package_TO_SOT_SMD:SOT-23, symbol Transistor_FET:AO3401A
- added R26: 1k, Resistor_SMD:R_0402_1005Metric, symbol Device:R
- added R27: 10k, Resistor_SMD:R_0402_1005Metric, symbol Device:R
Connections:
- net 3V3: now also R27.2
- net at U1.29 (SD3/IO10): now also R26.1, R27.1
- net at C20.2, L2.2: now also Q1.2 (S); no longer U5.7 (VCC_IO), U5.8 (VCC)
- new net: Q1.3 (D), U5.7 (VCC_IO), U5.8 (VCC)
- new net Pnp_Gps: Q1.1 (G), R26.2
Other:
- moved on the sheet: C16, C20, L2, R19

Commit message: Varicela y footpads
Parts:
- added TP10, TP11, TP2, TP3, TP4, TP5, TP6, TP7, TP8, TP9: TestPoint, TestPoint:TestPoint_Pad_1.0x1.0mm, symbol Connector:TestPoint
Connections:
- net +BATT: now also TP3.1
- net 3V3: now also TP4.1, TP5.1, TP7.1
- net ECHO_Sensor: now also TP10.1
- net PWR_Sensor: now also TP11.1
- net TRIG_Sensor: now also TP9.1
- net VBUS: now also TP2.1
- net uC_EN: now also TP6.1
- net at Q1.3 (D), U5.7 (VCC_IO), U5.8 (VCC): now also TP8.1

Commit message: Add files via upload
Parts:
- C10, C12, C13: value 100n -> 0.1u
Connections:
- net GND: now also U4.17 (VSS), U4.8 (VSS)
- net VBUS: no longer U4.17 (VSS), U4.8 (VSS)
Changed lines of the file:
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@@
 	)
 	(junction
-		(at 110.49 154.94)
-		(diameter 0)
-		(color 0 0 0 0)
-	)
-	(junction
 		(at 262.89 146.05)
 		(diameter 0)
@@
 	(wire
 		(pts
-			(xy 110.49 154.94) (xy 110.49 160.02)
-		)
-		(stroke
-			(width 0)
-			(type default)
-		)
-	)
-	(wire
-		(pts
 			(xy 74.93 92.71) (xy 80.01 92.71)
 		)
@@
 	(wire
 		(pts
+			(xy 102.87 156.21) (xy 106.68 156.21)
+		)
+		(stroke
+			(width 0)
+			(type default)
+		)
+	)
+	(wire
+		(pts
 			(xy 254 165.1) (xy 261.62 165.1)
 		)
@@
 		)
 	)
+	(wire
+		(pts
+			(xy 110.49 160.02) (xy 106.68 160.02)
+		)
+		(stroke
+			(width 0)
+			(type default)
+		)
+	)
 	(polyline
 		(pts
@@
 	(wire
 		(pts
+			(xy 106.68 160.02) (xy 106.68 156.21)
+		)
+		(stroke
+			(width 0)
+			(type default)
+		)
+	)
+	(wire
+		(pts
 			(xy 74.93 35.56) (xy 62.23 35.56)
 		)
@@
 			)
 		)
-		(property "Value" "100n"
+		(property "Value" "0.1u"
 			(at 255.27 152.3999 0)
 			(effects
@@
 			)
 		)
-		(property "Value" "100n"
+		(property "Value" "0.1u"
 			(at 266.7 152.3999 0)
 			(effects
@@
 	)
 	(symbol
+		(lib_id "power:GND")
+		(at 102.87 156.21 0)
+		(unit 1)
+		(exclude_from_sim no)
+		(in_bom yes)
+		(on_board yes)
+		(dnp no)
+		(fields_autoplaced yes)
+		(property "Reference" "#PWR036"
+			(at 102.87 162.56 0)
+			(effects
+				(font
+					(size 1.27 1.27)
+				)
+				(hide yes)
+			)
+		)
+		(property "Value" "GND"
+			(at 102.87 161.29 0)
+			(effects
+				(font
+					(size 1.27 1.27)
+				)
+			)
+		)
+		(property "Footprint" ""
+			(at 102.87 156.21 0)
+			(effects
+				(font
+					(size 1.27 1.27)
+				)
+				(hide yes)
+			)
+		)
+		(property "Datasheet" ""
+			(at 102.87 156.21 0)
+			(effects
+				(font
+					(size 1.27 1.27)
+				)
+				(hide yes)
+			)
+		)
+		(property "Description" "Power symbol creates a global label with name \"GND\" , ground"
+			(at 102.87 156.21 0)
+			(effects
+				(font
+					(size 1.27 1.27)
+				)
+				(hide yes)
+			)
+		)
+		(pin "1"
+		)
+		(instances
+			(project ""
+				(path "/80d6a340-3f89-493a-85f7-c642314f6a81"
+					(reference "#PWR036")
+					(unit 1)
+				)
+			)
+		)
+	)
+	(symbol
 		(lib_id "Device:R")
 		(at 127 82.55 0)
@@
 			)
 		)
-		(property "Value" "100n"
+		(property "Value" "0.1u"
 			(at 280.67 152.3999 0)
 			(effects
