File: PcbArroz.kicad_pcb (KiCad board)
At the start: 4 copper layers, 88 x 33 mm, 62 parts, among them J1 Conn_Coaxial_Small, J2 USB_C_Receptacle_USB2.0_16P, Q2 SS8050, Q3 AO3400A, Q4 SS8050, SW1 SW_Push, SW2 SW_SPST, U1 ESP32-PICO-D4, U2 RFM95W-915S2, U3 TPS62A01ADRL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

Commit message: V1 + via rules .3mm
Routing:
- net GND: track 21.6 -> 22.2 mm
Changed lines of the file:
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@@
+	)
+	(segment
+		(start 205.3818 154.2346)
+		(end 205.3818 154.0103)
+		(width 0.2)
+		(layer "F.Cu")
+		(net 5)
 	)
 	(segment
@@
 	)
 	(segment
-		(start 205.0626 153.6403)
-		(end 205.0626 153.6911)
-		(width 0.5)
-		(layer "F.Cu")
-		(net 5)
-	)
-	(segment
 		(start 210.7432 144.4772)
 		(end 210.8474 144.373)
@@
 	)
 	(segment
+		(start 206.4596 149.2715)
+		(end 206.7136 149.0175)
+		(width 0.5)
+		(layer "F.Cu")
+		(net 5)
+	)
+	(segment
+		(start 210.778002 139.9276)
+		(end 211.2063 139.9276)
+		(width 0.2)
+		(layer "F.Cu")
+		(net 5)
+	)
+	(segment
+		(start 203.1635 152.6946)
+		(end 202.3818 152.6946)
+		(width 0.3)
+		(layer "F.Cu")
+		(net 5)
+	)
+	(segment
+		(start 198.1148 137.2148)
+		(end 196.7648 137.2148)
+		(width 0.5)
+		(layer "F.Cu")
+		(net 5)
+	)
+	(segment
+		(start 241.431 152.402)
+		(end 241.431 151.8686)
+		(width 0.5)
+		(layer "F.Cu")
+		(net 5)
+	)
+	(segment
+		(start 241.431 151.8686)
+		(end 241.431 151.386)
+		(width 0.5)
+		(layer "F.Cu")
+		(net 5)
+	)
+	(segment
+		(start 203.8473 151.8693)
+		(end 203.8473 152.0108)
+		(width 0.3)
+		(layer "F.Cu")
+		(net 5)
+	)
+	(segment
+		(start 208.945 142.623)
+		(end 209.0466 142.5214)
+		(width 0.2)
+		(layer "F.Cu")
+		(net 5)
+	)
+	(segment
+		(start 216.1734 148.3367)
+		(end 216.9421 148.3367)
+		(width 0.2)
+		(layer "F.Cu")
+		(net 5)
+	)
+	(segment
+		(start 206.4451 149.2715)
+		(end 206.4596 149.2715)
+		(width 0.5)
+		(layer "F.Cu")
+		(net 5)
+	)
+	(segment
+		(start 208.9958 141.5308)
+		(end 209.0212 141.5054)
+		(width 0.2)
+		(layer "F.Cu")
+		(net 5)
+	)
+	(segment
+		(start 204.1318 140.05869)
+		(end 203.77729 140.4132)
+		(width 0.3)
+		(layer "F.Cu")
+		(net 5)
+	)
+	(segment
+		(start 205.3818 154.0103)
+		(end 205.0348 153.6633)
+		(width 0.2)
+		(layer "F.Cu")
+		(net 5)
+	)
+	(segment
+		(start 210.085002 139.2346)
+		(end 210.778002 139.9276)
+		(width 0.2)
+		(layer "F.Cu")
+		(net 5)
+	)
+	(segment
 		(start 205.0348 153.6633)
 		(end 205.0348 152.5568)
-		(width 0.2)
-		(layer "F.Cu")
-		(net 5)
-	)
-	(segment
-		(start 206.4596 149.2715)
-		(end 206.7136 149.0175)
-		(width 0.5)
-		(layer "F.Cu")
-		(net 5)
-	)
-	(segment
-		(start 210.778002 139.9276)
-		(end 211.2063 139.9276)
-		(width 0.2)
-		(layer "F.Cu")
-		(net 5)
-	)
-	(segment
-		(start 203.1635 152.6946)
-		(end 202.3818 152.6946)
-		(width 0.3)
-		(layer "F.Cu")
-		(net 5)
-	)
-	(segment
-		(start 198.1148 137.2148)
-		(end 196.7648 137.2148)
-		(width 0.5)
-		(layer "F.Cu")
-		(net 5)
-	)
-	(segment
-		(start 241.431 152.402)
-		(end 241.431 151.8686)
-		(width 0.5)
-		(layer "F.Cu")
-		(net 5)
-	)
-	(segment
-		(start 241.431 151.8686)
-		(end 241.431 151.386)
-		(width 0.5)
-		(layer "F.Cu")
-		(net 5)
-	)
-	(segment
-		(start 203.8473 151.8693)
-		(end 203.8473 152.0108)
-		(width 0.3)
-		(layer "F.Cu")
-		(net 5)
-	)
-	(segment
-		(start 208.945 142.623)
-		(end 209.0466 142.5214)
-		(width 0.2)
-		(layer "F.Cu")
-		(net 5)
-	)
-	(segment
-		(start 216.1734 148.3367)
-		(end 216.9421 148.3367)
-		(width 0.2)
-		(layer "F.Cu")
-		(net 5)
-	)
-	(segment
-		(start 206.4451 149.2715)
-		(end 206.4596 149.2715)
-		(width 0.5)
-		(layer "F.Cu")
-		(net 5)
-	)
-	(segment
-		(start 208.9958 141.5308)
-		(end 209.0212 141.5054)
-		(width 0.2)
-		(layer "F.Cu")
-		(net 5)
-	)
-	(segment
-		(start 204.1318 140.05869)
-		(end 203.77729 140.4132)
-		(width 0.3)
-		(layer "F.Cu")
-		(net 5)
-	)
-	(segment
-		(start 205.0626 153.6911)
-		(end 205.0348 153.6633)
-		(width 0.2)
-		(layer "F.Cu")
-		(net 5)
-	)
-	(segment
-		(start 210.085002 139.2346)
-		(end 210.778002 139.9276)
 		(width 0.2)
 		(layer "F.Cu")
@@
 		(at 201.6042 149.1953)
 		(size 0.5)
-		(drill 0.2)
+		(drill 0.3)
 		(layers "F.Cu" "B.Cu")
 		(net 5)
@@
 	(via
 		(at 202.3818 152.6946)
-		(size 0.5)
-		(drill 0.2)
+		(size 0.6)
+		(drill 0.3)
 		(layers "F.Cu" "B.Cu")
 		(net 5)
@@
 	)
 	(via
-		(at 205.0626 153.6911)
-		(size 0.5)
-		(drill 0.2)
+		(at 205.3818 154.2346)
+		(size 0.6)
+		(drill 0.3)
 		(layers "F.Cu" "B.Cu")
 		(net 5)
@@
 		(at 200.8672 138.8892)
 		(size 0.5)
-		(drill 0.2)
+		(drill 0.3)
 		(layers "F.Cu" "B.Cu")
 		(net 5)
@@
 		(at 203.945 147.2863)
 		(size 0.5)
-		(drill 0.2)
-		(layers "F.Cu" "B.Cu")
-		(net 5)
+		(drill 0.3)
+		(layers "F.Cu" "B.Cu")
+		(net 5)

Commit message: agregados pads
Parts:
- added TP1: TestPoint, TestPoint:TestPoint_Pad_1.0x1.0mm, F.Cu at (201.2, 146.6)
- added TP10: TestPoint, TestPoint:TestPoint_Pad_1.0x1.0mm, F.Cu at (237.3, 150.6)
- added TP2: TestPoint, TestPoint:TestPoint_Pad_1.0x1.0mm, F.Cu at (218.7, 146.9)
- added TP3: TestPoint, TestPoint:TestPoint_Pad_1.0x1.0mm, F.Cu at (205.6, 136.2)
- added TP4: TestPoint, TestPoint:TestPoint_Pad_1.0x1.0mm, F.Cu at (222.0, 133.1)
- added TP5: TestPoint, TestPoint:TestPoint_Pad_1.0x1.0mm, F.Cu at (209.3, 144.0)
- added TP7: TestPoint, TestPoint:TestPoint_Pad_1.0x1.0mm, F.Cu at (237.1, 141.0)
- added TP8: TestPoint, TestPoint:TestPoint_Pad_1.0x1.0mm, F.Cu at (223.1, 159.6)
- added TP9: TestPoint, TestPoint:TestPoint_Pad_1.0x1.0mm, F.Cu at (220.6, 159.6)
- C3: moved to B.Cu
- moved C3 2.46 mm to (238.3, 150.6)
- moved R18 0.88 mm to (238.1, 148.7)
- moved C9 0.87 mm to (202.2, 151.4)
Routing:
- net +3.3V: track 52.0 -> 67.5 mm, vias 15 -> 19
- net GND: track 22.2 -> 33.0 mm, vias 76 -> 82
- net Net-(BT2-+): track 32.9 -> 36.0 mm
- net ECHO_Sensor: track 20.2 -> 22.8 mm
- net TRIG_Sensor: track 23.8 -> 26.2 mm
- net VBUS: track 50.5 -> 52.2 mm
- net +BATT: track 27.1 -> 25.4 mm
- net NSS_LoRa: track 13.3 -> 12.1 mm
- net Reset_LoRa: track 10.5 -> 9.59 mm
- net uC_EN: track 34.4 -> 34.9 mm
Other:
- board text added: "5V"
- board text added: "GND"
