File: PcbArroz.kicad_sch (KiCad schematic)
At the start: 57 parts, among them J1 Conn_Coaxial_Small, J2 USB_C_Receptacle_USB2.0_16P, Q2 SS8050, Q3 AO3400A, Q4 SS8050, SW1 SW_Push, U1 ESP32-PICO-D4, U2 RFM95W-915S2, U3 TPS62A01ADRL, U4 BQ24074RGT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

Commit message: Revision general pcb
Connections:
- net USB_D+: now also J2.A6 (D+), J2.B6 (D+), U7.1 (I/O1)
- net USB_D-: now also J2.A7 (D-), J2.B7 (D-), U7.3 (I/O2)
Changed lines of the file:
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@@
 		)
 	)
+	(label "D+"
+		(at 40.64 226.06 0)
+		(effects
+			(font
+				(size 1.27 1.27)
+			)
+			(justify left bottom)
+		)
+	)
+	(label "D+"
+		(at 58.42 226.06 0)
+		(effects
+			(font
+				(size 1.27 1.27)
+			)
+			(justify left bottom)
+		)
+	)
+	(label "D-"
+		(at 58.42 223.52 0)
+		(effects
+			(font
+				(size 1.27 1.27)
+			)
+			(justify left bottom)
+		)
+	)
+	(label "D-"
+		(at 40.64 223.52 0)
+		(effects
+			(font
+				(size 1.27 1.27)
+			)
+			(justify left bottom)
+		)
+	)
 	(global_label "3V3"
 		(shape output)
@@
 		(on_board yes)
 		(dnp no)
-		(fields_autoplaced yes)
 		(property "Reference" "C14"
 			(at 41.91 38.0999 0)
@@
 		(on_board yes)
 		(dnp no)
-		(fields_autoplaced yes)
 		(property "Reference" "R10"
 			(at 125.73 238.7599 0)

Commit message: Pcb v1
Parts:
- added SW2: SW_SPST, Button_Switch_THT:SW_DIP_SPSTx01_Slide_6.7x4.1mm_W7.62mm_P2.54mm_LowProfile, symbol Switch:SW_SPST
Connections:
- net 3V3 is gone; now on net +3.3V: AJ-SR04M1.1 (5V), C1.1, C7.1, D3.2 (A), L1.2, R4.1, U2.13 (3.3V)
- net +BATT: now also SW2.1 (A); no longer BT2.1 (+)
- new net: BT2.1 (+), SW2.2 (B)
Other:
- moved on the sheet: BT2
Changed lines of the file:
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@@
 	(wire
 		(pts
-			(xy 146.05 148.59) (xy 146.05 151.13)
+			(xy 146.05 149.86) (xy 146.05 151.13)
 		)
 		(stroke
@@
 	(wire
 		(pts
-			(xy 60.96 257.81) (xy 66.04 257.81)
+			(xy 60.96 257.81) (xy 77.47 257.81)
 		)
 		(stroke
@@
 	(wire
 		(pts
-			(xy 66.04 257.81) (xy 66.04 255.27)
+			(xy 77.47 257.81) (xy 77.47 254)
 		)
 		(stroke
@@
 	(wire
 		(pts
-			(xy 66.04 246.38) (xy 66.04 247.65)
-		)
-		(stroke
-			(width 0)
-			(type default)
-		)
-	)
-	(wire
-		(pts
 			(xy 234.95 196.85) (xy 234.95 208.28)
 		)
@@
 	(wire
 		(pts
+			(xy 77.47 246.38) (xy 76.2 246.38)
+		)
+		(stroke
+			(width 0)
+			(type default)
+		)
+	)
+	(wire
+		(pts
 			(xy 312.42 228.6) (xy 317.5 228.6)
 		)
@@
 		)
 	)
-	(global_label "3V3"
+	(global_label "+3.3V"
 		(shape output)
 		(at 182.88 256.54 0)
@@
 		)
 		(property "Intersheetrefs" "${INTERSHEET_REFS}"
-			(at 189.3728 256.54 0)
+			(at 191.55 256.54 0)
 			(effects
 				(font
@@
 		)
 	)
-	(global_label "3V3"
+	(global_label "+3.3V"
 		(shape input)
 		(at 63.5 147.32 90)
@@
 		)
 		(property "Intersheetrefs" "${INTERSHEET_REFS}"
-			(at 63.5 140.8272 90)
+			(at 63.5 138.65 90)
 			(effects
 				(font
@@
 		)
 	)
-	(global_label "3V3"
+	(global_label "+3.3V"
 		(shape input)
-		(at 146.05 148.59 90)
+		(at 146.05 149.86 90)
 		(fields_autoplaced yes)
 		(effects
@@
 		)
 		(property "Intersheetrefs" "${INTERSHEET_REFS}"
-			(at 146.05 142.0972 90)
+			(at 146.05 141.19 90)
 			(effects
 				(font
@@
 		)
 		(property "Netclass" "Power"
-			(at 148.2408 148.59 90)
+			(at 148.2408 149.86 90)
 			(effects
 				(font
@@
 	(symbol
 		(lib_id "Device:Battery_Cell")
-		(at 66.04 252.73 0)
+		(at 77.47 251.46 0)
 		(unit 1)
 		(exclude_from_sim no)
@@
 		(on_board yes)
 		(dnp no)
-		(fields_autoplaced yes)
 		(property "Reference" "BT2"
-			(at 69.85 249.6184 0)
+			(at 81.788 248.666 0)
 			(effects
 				(font
@@
 		)
 		(property "Value" "Battery_Cell"
-			(at 69.85 252.1584 0)
+			(at 76.962 252.222 0)
 			(effects
 				(font
@@
 		)
 		(property "Footprint" "Connector_JST:JST_EH_S2B-EH_1x02_P2.50mm_Horizontal"
-			(at 66.04 251.206 90)
+			(at 77.47 249.936 90)
 			(effects
 				(font
@@
 		)
 		(property "Datasheet" "~"
-			(at 66.04 251.206 90)
+			(at 77.47 249.936 90)
 			(effects
 				(font
@@
 		)
 		(property "Description" "Single-cell battery"
-			(at 66.04 252.73 0)
+			(at 77.47 251.46 0)
 			(effects
 				(font
@@
 					(unit 1)
 				)
+			)
+		)
+	)
+	(symbol
+		(lib_id "Switch:SW_SPST")
+		(at 71.12 246.38 0)
+		(unit 1)
+		(exclude_from_sim no)
+		(in_bom yes)
+		(on_board yes)
+		(dnp no)
+		(property "Reference" "SW2"
+			(at 71.12 248.412 0)
+			(effects
+				(font
+					(size 1.27 1.27)
+				)
+			)
+		)
+		(property "Value" "SW_SPST"
+			(at 70.104 250.444 0)
+			(effects
+				(font
+					(size 1.27 1.27)
+				)
+			)
+		)
+		(property "Footprint" "Button_Switch_THT:SW_DIP_SPSTx01_Slide_6.7x4.1mm_W7.62mm_P2.54mm_LowProfile"
+			(at 71.12 246.38 0)
+			(effects
+				(font
+					(size 1.27 1.27)
+				)
+				(hide yes)
+			)
+		)
+		(property "Datasheet" "~"
+			(at 71.12 246.38 0)
+			(effects
+				(font
+					(size 1.27 1.27)
+				)
+				(hide yes)
+			)
+		)
+		(property "Description" "Single Pole Single Throw (SPST) switch"
+			(at 71.12 246.38 0)
+			(effects
+				(font
+					(size 1.27 1.27)
+				)
+				(hide yes)
+			)
+		)
+		(pin "2"
+		)
+		(pin "1"
+		)
+		(instances
+			(project ""
+				(path "/80d6a340-3f89-493a-85f7-c642314f6a81"
+					(reference "SW2")
+					(unit 1)
+				)

Commit message: agregados pads
Parts:
- added TP1, TP10, TP2, TP3, TP4, TP5, TP7, TP8, TP9: TestPoint, TestPoint:TestPoint_Pad_1.0x1.0mm, symbol Connector:TestPoint
Connections:
- net +3.3V: now also TP2.1, TP5.1, TP7.1
- net BOOT: now also TP10.1
- net ECHO_Sensor: now also TP8.1
- net GND: now also TP3.1
- net TRIG_Sensor: now also TP9.1
- net VBUS: now also TP1.1
- net uC_EN: now also TP4.1
