File: V3/V3/V3.kicad_sch (KiCad schematic)
At the start: 77 parts, among them J1 USB_C_Receptacle_USB2.0_16P, J2 Conn_Coaxial_Small, J4 Conn_Coaxial_Small, Q1 AO3401, Q2 AO3401A, Q3 AO3400A, SW1 SW_Push, SW2 SW_Push, U1 CP2102, U3 ESP32-S3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

Commit message: 1
Parts:
- added R13: 1R, Resistor_SMD:R_0805_2012Metric, symbol Device:R
- 2n7002bks1: footprint (none) -> Package_TO_SOT_SMD:SOT-363_SC-70-6; LCSC (none) -> C68181
- AJ-SR04M1: footprint Connector_PinSocket_1.00mm:PinSocket_1x04_P1.00mm_Vertical -> Connector_PinHeader_2.54mm:PinHeader_1x04_P2.54mm_Vertical
- AP2112K-3.3TRG1: renamed from U2; footprint (none) -> Package_TO_SOT_SMD:SOT-23-5; LCSC (none) -> C23380830
- BT1: footprint (none) -> Connector_JST:JST_EH_S2B-EH_1x02_P2.50mm_Horizontal
- BT2: footprint CR1220 socket:BAT_1056TR -> Battery:BatteryHolder_Keystone_1057_1x2032; LCSC (none) -> C238068
- C1, C10, C11, C12, C13, C14, C15, C16, C17, C18, C19, C2, C20, C24, C3, C4, C5, C6, C7, C8, C9: footprint (none) -> Capacitor_SMD:C_0805_2012Metric
- C23: renamed from C11; footprint (none) -> Capacitor_SMD:C_0805_2012Metric
- C29: renamed from C15; footprint (none) -> Capacitor_SMD:C_0805_2012Metric
- C30: renamed from C23; footprint (none) -> Capacitor_SMD:C_0805_2012Metric
- D1: LCSC (none) -> C28646388
- D2: LCSC (none) -> C727114
- J1: LCSC (none) -> C7095263
- J2, J4: LCSC (none) -> C88373
- L1: footprint (none) -> Inductor_SMD:L_0402_1005Metric; LCSC (none) -> C18216
- L2: footprint (none) -> Inductor_SMD:L_0201_0603Metric; LCSC (none) -> C12099
- L3: footprint Inductor_SMD:L_0805_2012Metric -> Inductor_SMD:L_0603_1608Metric; LCSC (none) -> C12100
- LGS4056HDA1: footprint (none) -> Package_DFN_QFN:DFN-8-1EP_3x3mm_P0.5mm_EP1.7x2.4mm; LCSC (none) -> C5124109
- Q1: LCSC (none) -> AO3401
- Q2: LCSC (none) -> C15127
- Q3: LCSC (none) -> C20917
- R1, R10, R2, R24, R26, R27, R28, R29, R3, R4, R5, R7, R8: footprint (none) -> Resistor_SMD:R_0805_2012Metric
- R11, R12, R25, R6, R9: footprint Resistor_SMD:R_0402_1005Metric -> Resistor_SMD:R_0805_2012Metric
- SW1, SW2: footprint (none) -> Button_Switch_SMD:SW_SPST_PTS645Sx43SMTR92; LCSC (none) -> C49234152
- U1: LCSC (none) -> C6568
- U3: value ESP32-S3 -> ESP32-S3FN8; LCSC (none) -> C2913196
- Y1: footprint (none) -> Crystal:Crystal_SMD_3225-4Pin_3.2x2.5mm; LCSC (none) -> C5380316
- Y2: footprint (none) -> Crystal:Crystal_SMD_SeikoEpson_MC146-4Pin_6.7x1.5mm; LCSC (none) -> C15482
Connections:
- net GND: no longer BT1.1 (+), C5.1, Q1.3 (D)
- net MISO_LoRa: now also U4.3 (MOSI); no longer U4.2 (MISO)
- net MOSI_LoRa: now also U4.2 (MISO); no longer U4.3 (MOSI)
- net VDD_3V3: no longer U3.20 (VDD3P3_RTC)
- net VDD_5V: now also R13.2; no longer C9.1
- net at C17.1, C18.1: no longer U3.29 (VDD_SPI)
- new net: C9.1, R13.1
- new net VBAT: BT1.1 (+), C5.1, LGS4056HDA1. (BAT), Q1.3 (D)
Other:
- note added: "Alimentación y batería"
- moved on the sheet: C9

Commit message: falta rutear esp v3
Parts:
- BT2: footprint Battery:BatteryHolder_Keystone_1057_1x2032 -> Footprints:pila
- U2: renamed from LGS4056HDA1; value ~ -> LGS4056HDA1
- U5: footprint Teseo:ARRAY_LIV3R_STM -> Footprints:Teseo
- U6: renamed from AP2112K-3.3TRG1; value ~ -> AP2112K-3.3TRG1
- U8: renamed from 2n7002bks1; value ~ -> 2n7002bks1
Connections:
- net VDD_3v3 is gone; now on net VDD_3V3: R7.2
- net CHRG: now also U2.7 (CHRG); no longer U2. (BAT)
- net GND: now also U2.1 (Temp), U2.3 (Gnd), U2.6 (DONE), U6.2 (GND); no longer U2. (BAT), U6. (NC)
- net VBAT: now also U2.5 (BAT); no longer U2. (BAT)
- net VDD_3V3: now also U6.5 (OUT); no longer U6. (NC)
- net VDD_5V: now also U2.4 (Vcc), U2.8 (CE); no longer U2. (BAT)
- net at R24.2: now also U2.2 (Prog); no longer U2. (BAT)
- net at C8.1, D2.1 (K), Q1.2 (S)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: now also U6.1 (IN); no longer U6. (NC)
- net at R8.2: now also U6.3 (EN); no longer U6. (NC)
Changed lines of the file:
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@@
 		)
 	)
-	(global_label "VDD_3v3"
+	(global_label "VDD_3V3"
 		(shape input)
 		(at 29.21 278.13 180)
@@
 		)
 		(property "Intersheetrefs" "${INTERSHEET_REFS}"
-			(at 18.242 278.13 0)
+			(at 18.121 278.13 0)
 			(effects
 				(font
@@
 		(on_board yes)
 		(dnp no)
-		(property "Reference" "2n7002bks1"
+		(property "Reference" "U8"
 			(at 64.008 265.43 0)
 			(effects
@@
 			)
 		)
-		(property "Value" "~"
-			(at 63.5 251.46 0)
+		(property "Value" "2n7002bks1"
+			(at 63.5 270.764 0)
 			(effects
 				(font
@@
 			(project ""
 				(path "/f20c1557-6840-4cf5-bfcb-5ed671cb3443"
-					(reference "2n7002bks1")
+					(reference "U8")
 					(unit 1)
 				)
@@
 			)
 		)
-		(property "Footprint" "Teseo:ARRAY_LIV3R_STM"
+		(property "Footprint" "Footprints:Teseo"
 			(at 269.24 38.1 0)
 			(effects
@@
 		(on_board yes)
 		(dnp no)
-		(property "Reference" "AP2112K-3.3TRG1"
+		(property "Reference" "U6"
 			(at 112.014 33.274 0)
 			(effects
@@
 			)
 		)
-		(property "Value" "~"
+		(property "Value" "AP2112K-3.3TRG1"
 			(at 112.395 31.75 0)
 			(effects
@@
 			)
 		)
-		(pin ""
+		(pin "3"
 		)
-		(pin ""
+		(pin "5"
 		)
-		(pin ""
+		(pin "4"
 		)
-		(pin ""
+		(pin "1"
 		)
-		(pin ""
+		(pin "2"
 		)
 		(instances
 			(project ""
 				(path "/f20c1557-6840-4cf5-bfcb-5ed671cb3443"
-					(reference "AP2112K-3.3TRG1")
+					(reference "U6")
 					(unit 1)
 				)
@@
 		(dnp no)
 		(fields_autoplaced yes)
-		(property "Reference" "LGS4056HDA1"
+		(property "Reference" "U2"
 			(at 105.41 73.6599 90)
 			(effects
@@
 			)
 		)
-		(property "Value" "~"
+		(property "Value" "LGS4056HDA1"
 			(at 105.41 76.1999 90)
 			(effects
@@
 			)
 		)
-		(pin ""
+		(pin "4"
 		)
-		(pin ""
+		(pin "3"
 		)
-		(pin ""
+		(pin "5"
 		)
-		(pin ""
+		(pin "8"
 		)
-		(pin ""
+		(pin "6"
 		)
-		(pin ""
+		(pin "1"
 		)
-		(pin ""
+		(pin "2"
 		)
-		(pin ""
+		(pin "7"
 		)
 		(instances
 			(project ""
 				(path "/f20c1557-6840-4cf5-bfcb-5ed671cb3443"
-					(reference "LGS4056HDA1")
+					(reference "U2")
 					(unit 1)
 				)
@@
 			)
 		)
-		(property "Footprint" "Battery:BatteryHolder_Keystone_1057_1x2032"
+		(property "Footprint" "Footprints:pila"
 			(at 365.76 69.85 0)
 			(effects
