File: Version 3.0/V3/V3.kicad_pcb (KiCad board)
At the start: 4 copper layers, 78 parts, among them J1 USB_C_Receptacle_USB2.0_16P, J2 Conn_Coaxial_Small, J4 Conn_Coaxial_Small, Q1 AO3401, Q2 AO3401A, Q3 AO3400A, SW1 SW_Push, SW2 SW_Push, U1 CP2102, U2 LGS4056HDA1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

Commit message: V3 para revisar
Parts:
- D1: footprint Package_SON:WSON-6-1EP_2x2mm_P0.65mm_EP1x1.6mm -> Diode_SMD:D_SOD-523
- D2: footprint Diode_THT:D_DO-41_SOD81_P10.16mm_Horizontal -> Diode_SMD:D_SOD-323
- U8: value 2n7002bks1 -> 2n7002bks
- moved C28 115.2 mm to (110.8, 89.5), turned to -90 degrees
- moved J2 110.8 mm to (121.2, 96.3)
- moved C23 109.1 mm to (88.0, 103.5)
- moved U4 106.5 mm to (100.0, 88.8)
- moved TP10 106.2 mm to (94.8, 105.2)
- moved BT2 105.5 mm to (106.3, 68.2)
- moved C15 105.5 mm to (81.0, 100.5), turned to 90 degrees
- moved TP9 103.9 mm to (91.0, 101.2)
- moved C24 103.3 mm to (83.8, 101.8)
- moved Q3 101.4 mm to (95.5, 101.0)
- moved C30 93.4 mm to (78.0, 99.2)
- moved TP11 92.9 mm to (85.8, 97.5)
- moved C19 88.7 mm to (82.8, 93.8), turned to -90 degrees
- moved R6 88.5 mm to (89.2, 97.0), turned to 90 degrees
- moved AJ-SR04M1 88.1 mm to (101.7, 102.0), turned to 90 degrees
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Connections:
- C17 pad 1: Net-(C17-Pad1) -> Net-(U3-VDD_SPI)
- C18 pad 1: Net-(C17-Pad1) -> Net-(U3-VDD_SPI)
- C22 pad 1: 3V3 -> VDD_3V3
- C28 pad 1: 3V3 -> VDD_3V3
- D1 pad 2: GND -> VDD_5V
- L3 pad 1: 3V3 -> VDD_3V3
- R11 pad 1: Net-(U3-GPIO6) -> Net-(U3-GPIO35)
- R12 pad 1: Net-(U3-GPIO6) -> Net-(U3-GPIO35)
- U3 pad 10: AntOff_GPS -> PWR_Sensor
- U3 pad 11: Net-(U3-GPIO6) -> unconnected-(U3-GPIO6-Pad11)
- U3 pad 12: NSS_LoRa -> Reset_LoRa
- U3 pad 13: RX/TXdone_LoRa -> NSS_LoRa
- U3 pad 15: MOSI_LoRa -> MISO_LoRa
- U3 pad 16: MISO_LoRa -> MOSI_LoRa
- U3 pad 17: Reset_LoRa -> RX/TXdone_LoRa
- U3 pad 18: CADdetect_LoRa -> RXtimeout_LoRa
- U3 pad 19: RXtimeout_LoRa -> CADdetect_LoRa
- U3 pad 20: unconnected-(U3-VDD3P3_RTC-Pad20) -> VDD_3V3
- U3 pad 29: unconnected-(U3-VDD_SPI-Pad29) -> Net-(U3-VDD_SPI)
- U3 pad 38: PWR_Sensor -> Reset_GPS
- U3 pad 39: TRIG_Sensor -> AntOff_GPS
- U3 pad 40: ECHO_Sensor -> Net-(U3-GPIO35)
- U3 pad 41: Tx_GPS -> Rx_GPS
- U3 pad 42: Rx_GPS -> Tx_GPS
- U3 pad 8: unconnected-(U3-GPIO3-Pad8) -> ECHO_Sensor
- U3 pad 9: Reset_GPS -> TRIG_Sensor
- U4 pad 13: 3V3 -> VDD_3V3
Routing:
- net AntOff_GPS: track 0.00 -> 69.5 mm, vias 0 -> 2
- net Wake_GPS: track 0.00 -> 54.1 mm, vias 0 -> 2
- net Reset_GPS: track 0.00 -> 53.4 mm, vias 0 -> 2
- net CHIP_PU: track 4.26 -> 51.7 mm, vias 0 -> 2
- net VBatt: track 0.00 -> 46.7 mm, vias 0 -> 2
- net ECHO_Sensor: track 0.00 -> 43.4 mm
- net PPS_GPS: track 0.00 -> 40.6 mm, vias 0 -> 2
- net TRIG_Sensor: track 0.00 -> 39.9 mm
- net Rx_GPS: track 0.00 -> 36.5 mm
- net Tx_GPS: track 0.00 -> 35.6 mm
- net USER_KEY: track 25.5 -> 58.8 mm, vias 0 -> 2
- net RXtimeout_LoRa: track 0.00 -> 31.7 mm, vias 0 -> 2
- net RX/TXdone_LoRa: track 0.00 -> 31.6 mm, vias 0 -> 2
- net CADdetect_LoRa: track 0.00 -> 31.5 mm, vias 0 -> 2
- net VDD_3V3: track 14.8 -> 40.3 mm, vias 5 -> 14
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Other:
- board outline added: 90.8 x 60.5 mm
