File: Version 3.0/V3/V3.kicad_pcb (KiCad board)
At the start: 4 copper layers, 90.8 x 60.5 mm, 78 parts, among them J1 USB_C_Receptacle_USB2.0_16P, J2 Conn_Coaxial_Small, J4 Conn_Coaxial_Small, Q1 AO3401, Q2 AO3401A, Q3 AO3400A, SW1 SW_Push, SW2 SW_Push, U1 CP2102, U2 LGS4056HDA1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

Commit message: V3 final
Parts:
- added UCU: LOGO, logos:LogoUCU, B.Cu at (117.0, 78.4)
Connections:
- Y1 pad 2: XTAL_P -> (no net)
- Y1 pad 3: (no net) -> XTAL_P
- Y2 pad 2: 32K_XP -> (no net)
- Y2 pad 4: (no net) -> 32K_XP
Routing:
- net GND: track 40.1 -> 73.4 mm, vias 46 -> 59
- net XTAL_P: track 6.16 -> 9.16 mm, vias 1 -> 0
- net AntOff_GPS: track 69.5 -> 70.0 mm
- net XTAL_N: vias 1 -> 0
- net VDD_3V3: vias 14 -> 13
Other:
- board text added: "Arroz V3 CK, RDT, IR"

Commit message: Firmware Final
Parts:
- L2: footprint Inductor_SMD:L_0201_0603Metric -> Inductor_SMD:L_0603_1608Metric
- U2: footprint Package_DFN_QFN:DFN-8-1EP_3x3mm_P0.5mm_EP1.7x2.4mm -> Package_DFN_QFN:DFN-8-1EP_2x2mm_P0.5mm_EP0.6x1.2mm
- moved Y1 1.35 mm to (67.8, 96.2)
- moved L2 0.76 mm to (68.3, 92.5)
Connections:
- Y1 pad 1: XTAL_N -> XTAL_P
- Y1 pad 3: XTAL_P -> XTAL_N
Routing:
- net XTAL_N: track 20.3 -> 14.0 mm
- net GND: track 73.4 -> 74.9 mm
- net VDD_5V: track 92.9 -> 93.9 mm
- net Net-(U2-Prog): track 6.21 -> 6.71 mm
- net VBAT: track 27.7 -> 28.2 mm
