File: Version 3.0/V3/V3.kicad_sch (KiCad schematic)
At the start: 78 parts, among them J1 USB_C_Receptacle_USB2.0_16P, J2 Conn_Coaxial_Small, J4 Conn_Coaxial_Small, Q1 AO3401, Q2 AO3401A, Q3 AO3400A, SW1 SW_Push, SW2 SW_Push, U1 CP2102, U2 LGS4056HDA1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

Commit message: v3 para revisar
Parts:
- R3: now left out of the parts list
Connections:
- net AntOff_GPS: now also U3.39 (GPIO34); no longer U3.10 (GPIO5)
- net CADdetect_LoRa: now also U3.19 (GPIO14); no longer U3.18 (GPIO13)
- net ECHO_Sensor: now also U3.8 (GPIO3); no longer U3.40 (GPIO35)
- net MISO_LoRa: now also U3.15 (GPIO10); no longer U3.16 (GPIO11)
- net MOSI_LoRa: now also U3.16 (GPIO11); no longer U3.15 (GPIO10)
- net NSS_LoRa: now also U3.13 (GPIO8); no longer U3.12 (GPIO7)
- net PWR_Sensor: now also U3.10 (GPIO5); no longer U3.38 (GPIO33)
- net RXtimeout_LoRa: now also U3.18 (GPIO13); no longer U3.19 (GPIO14)
- net RX/TXdone_LoRa: now also U3.17 (GPIO12); no longer U3.13 (GPIO8)
- net Reset_GPS: now also U3.38 (GPIO33); no longer U3.9 (GPIO4)
- net Reset_LoRa: now also U3.12 (GPIO7); no longer U3.17 (GPIO12)
- net Rx_GPS: now also U3.41 (GPIO36); no longer U3.42 (GPIO37)
- net TRIG_Sensor: now also U3.9 (GPIO4); no longer U3.39 (GPIO34)
- net Tx_GPS: now also U3.42 (GPIO37); no longer U3.41 (GPIO36)
- net VDD_3V3: now also U3.20 (VDD3P3_RTC)
- net at R11.1, R12.1: now also U3.40 (GPIO35); no longer U3.11 (GPIO6)
- net at U3.29 (VDD_SPI): now also C17.1, C18.1
Other:
- moved on the sheet: R11, R12

Commit message: V3 para revisar
Parts:
- removed D1: RSB6.8S, Package_SON:WSON-6-1EP_2x2mm_P0.65mm_EP1x1.6mm, symbol Power_Protection:TVS1800DRV
- added D1: RSB6.8S, Diode_SMD:D_SOD-523, symbol Device:D
- AJ-SR04M1: LCSC (none) -> C7243
- D2: footprint Diode_THT:D_DO-41_SOD81_P10.16mm_Horizontal -> Diode_SMD:D_SOD-323
- Q1: LCSC AO3401 -> C181091
- U8: value 2n7002bks1 -> 2n7002bks
Connections:
- net 3V3 is gone; now on net VDD_3V3: C22.1, C28.1, L3.1, U4.13 (3.3V)
- net GND: now also D1.1 (K)
- net VDD_5V: now also D1.2 (A)
Other:
- moved on the sheet: J1, R26, R27, R28, R29
