File: Version 3.0/V3/V3.kicad_sch (KiCad schematic)
At the start: 78 parts, among them J1 USB_C_Receptacle_USB2.0_16P, J2 Conn_Coaxial_Small, J4 Conn_Coaxial_Small, Q1 AO3401, Q2 AO3401A, Q3 AO3400A, SW1 SW_Push, SW2 SW_Push, U1 CP2102, U2 LGS4056HDA1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

Commit message: Nodered
Parts:
- added C31: 10nF, Capacitor_SMD:C_0805_2012Metric, symbol Device:C
- added C32: 56pF, Capacitor_SMD:C_0603_1608Metric, symbol Device:C
- added L4: 27nH, Inductor_SMD:L_0603_1608Metric, symbol Device:L
- added Q4: AO3401A, Package_TO_SOT_SMD:SOT-23, symbol Transistor_FET:AO3401A
- added R14: 10k, Resistor_SMD:R_0805_2012Metric, symbol Device:R
- added R15: 1k, Resistor_SMD:R_0805_2012Metric, symbol Device:R
- added TP1: TestPoint, TestPoint:TestPoint_Pad_1.0x1.0mm, symbol Connector:TestPoint
Connections:
- net GND: now also C31.2, C32.1
- net Pnp_Gps: now also Q4.1 (G), R15.2
- net VDD_3V3: now also C31.1, L4.1, R14.2
- new net: C32.2, L4.2, Q4.2 (S)
- new net: Q4.3 (D), TP1.1
- new net GPIO35: R14.1, R15.1
