File: V3.0/V3/V3.kicad_sch (KiCad schematic)
At the start: 85 parts, among them J1 USB_C_Receptacle_USB2.0_16P, J2 Conn_Coaxial_Small, J4 Conn_Coaxial_Small, Q1 AO3401, Q2 AO3401A, Q3 AO3400A, Q4 AO3401A, SW1 SW_Push, SW2 SW_Push, U1 CP2102, U2 LGS4056HDA1, U3 ESP32-S3FN8, U4 RFM95W-915S2, U5 TESEO-LIV3R, U6 AP2112K-3.3TRG1, U8 2n7002bks, Y1 Crystal 40MHz/10ppm, Y2 32.768KHz/ESR≤70KΩ

Commit message: imagenes
Parts:
- removed C31: 10nF, Capacitor_SMD:C_0805_2012Metric, symbol Device:C
- removed C32: 56pF, Capacitor_SMD:C_0603_1608Metric, symbol Device:C
- removed L4: 27nH, Inductor_SMD:L_0603_1608Metric, symbol Device:L
- removed Q4: AO3401A, Package_TO_SOT_SMD:SOT-23, symbol Transistor_FET:AO3401A
- removed R14: 10k, Resistor_SMD:R_0805_2012Metric, symbol Device:R
- removed R15: 1k, Resistor_SMD:R_0805_2012Metric, symbol Device:R
- removed TP1: TestPoint, TestPoint:TestPoint_Pad_1.0x1.0mm, symbol Connector:TestPoint
Other:
- note added: "ESP32"
- note added: "USB TO UART"
- moved on the sheet: AJ-SR04M1, BT2, C11, C12, C13, C14, C15, C16, C17, C18, C19, C20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
